Commit message: framework world flange and place update

File: framework/urdf/ur10e_robotiq85_position.urdf (robot description, URDF)
Before this commit: robot ur10e_robotiq85_flange, 21 links, 20 joints
Links:
- removed link flange_link
Joints:
- removed joint flange-robotiq_85_base_joint
- removed joint robot_tool0-flange_joint
- added joint robot_tool0-robotiq_85_base_link: type fixed, parent robot_tool0, child gripper_robotiq_85_base_link, origin xyz=0 0 0 rpy=0 -1.57079632679 1.57079632679

File: framework_flange/urdf/ur10e_robotiq85_flange.urdf (robot description, URDF)
Before this commit: robot ur10e_robotiq85_flange, 21 links, 20 joints
Links:
- link flange_link: geometry collision mesh filename=package://ur10e_85_flange_moveit/flange/adapter.stl scale=0.025 0.025 0.025; visual mesh filename=package://ur10e_85_flange_moveit/flange/adapter.stl scale=0.025 0.025 0.025
Joints:
- joint flange-robotiq_85_base_joint: origin xyz=0 0 0.025 rpy=0 -1.57079632679 1.57079632679 -> xyz=0 0 0.08 rpy=0 -1.57079632679 1.57079632679
- joint robot_tool0-flange_joint: origin xyz=0 0 0.025 rpy=0 0 0 -> xyz=0 0 0.0 rpy=0 0 0

File: framework_switch/urdf/ur10e_robotiq85_switch.urdf (robot description, URDF)
Before this commit: robot ur10e_robotiq85_flange, 21 links, 20 joints
Links:
- removed link flange_link
- added link left_inner_finger_pad; collision box size=0.022 0.00635 0.05; visual box size=0.022 0.00635 0.05
- added link right_inner_finger_pad; collision box size=0.022 0.00635 0.05; visual box size=0.022 0.00635 0.05
- link gripper_robotiq_85_left_finger_tip_link: geometry collision mesh filename=package://cable_simulation/meshes/collision/robotiq_arg2f_8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 scale=0.001 0.001 0.001; visual mesh filename=package://cable_simulation/meshes/visual/robotiq_arg2f_85_i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 scale=0.001 0.001 0.001
- link gripper_robotiq_85_right_finger_tip_link: geometry collision mesh filename=package://cable_simulation/meshes/collision/robotiq_arg2f_8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 scale=0.001 0.001 0.001; visual mesh filename=package://cable_simulation/meshes/visual/robotiq_arg2f_85_i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 scale=0.001 0.001 0.001
Joints:
- removed joint flange-robotiq_85_base_joint
- removed joint robot_tool0-flange_joint
- added joint left_inner_finger_pad_joint: type fixed, parent gripper_robotiq_85_left_finger_tip_link, child left_inner_finger_pad, origin xyz=0.03175 0.0035 0 rpy=0 0 0, axis 0 0 1
- added joint right_inner_finger_pad_joint: type fixed, parent gripper_robotiq_85_right_finger_tip_link, child right_inner_finger_pad, origin xyz=0.03175 0.0035 0 rpy=0 0 0, axis 0 0 1
- added joint robot_tool0-robotiq_85_base_link: type fixed, parent robot_tool0, child gripper_robotiq_85_base_link, origin xyz=0 0 0 rpy=0 -1.57079632679 1.57079632679
