Commit message: xacro urdf clean up

File: framework/urdf/ur10e_robotiq85.xacro (robot description, xacro)
@@ -17,9 +17,9 @@
   <!-- define the ur10's position and orientation in the world coordinate system -->
     <link name="world"/>
+    <!-- TODO: check base_link name of robot -->
     <joint name="world_joint" type="fixed">
-    <parent link="world"/>
-    <child link="robot_base_link"/>
-    <!-- TODO: check base_link name of robot -->
-    <origin rpy="0.0 0.0 0.0" xyz="0.0 0.0 0.0"/>
+      <parent link="world"/>
+      <child link="robot_base_link"/>
+      <origin rpy="0.0 0.0 0.0" xyz="0.0 0.0 0.0"/>
     </joint>
   <gazebo>

File: framework_flange/urdf/ur10e_robotiq85_flange.xacro (robot description, xacro)
@@ -30,9 +30,9 @@
   <!-- define the ur10's position and orientation in the world coordinate system -->
     <link name="world"/>
+    <!-- TODO: check base_link name of robot -->
     <joint name="world_joint" type="fixed">
-    <parent link="world"/>
-    <child link="robot_base_link"/>
-    <!-- TODO: check base_link name of robot -->
-    <origin rpy="0.0 0.0 0.0" xyz="0.0 0.0 0.0"/>
+      <parent link="world"/>
+      <child link="robot_base_link"/>
+      <origin rpy="0.0 0.0 0.0" xyz="0.0 0.0 0.0"/>
     </joint>
  </xacro:macro>
